Commit message: added package for obj_detection and added 3d SLAM using rtab_map to fuse lidar + rgbd and visualize rgb measurements in rviz + slam_toolbox for 2d map

File: src/dog_utilities/urdf/go2_with_realsense.urdf (robot description, URDF)
Before this commit: robot go2, 34 links, 33 joints
Links:
- added link camera_color_optical_frame
Joints:
- added joint camera_color_optical_joint: type fixed, parent camera_link, child camera_color_optical_frame, origin xyz=0 0 0 rpy=-1.5708 0 -1.5708
